File: D21SequansAdapterBoard.kicad_pcb (KiCad board)
At the start: 4 copper layers, 80 x 82.1 mm, 14 parts, among them J1 Conn_02x18_Odd_Even, J2 Conn_02x20_Odd_Even, J3 Conn_01x24, J4 Conn_01x24, J5 Conn_01x24, J6 Conn_01x24

Commit message: layout complete
Parts:
- added Q1: MMBT3904, Package_TO_SOT_SMD:SOT-23, F.Cu at (137.4, 68.6)
- added Q2: MMBT3904, Package_TO_SOT_SMD:SOT-23, F.Cu at (137.4, 73.9)
- added Q3: MMBT3904, Package_TO_SOT_SMD:SOT-23, F.Cu at (137.4, 79.2)
- added Q4: MMBT3904, Package_TO_SOT_SMD:SOT-23, F.Cu at (137.8, 84.2)
- added R5: 100, Resistor_SMD:R_0603_1608Metric_Pad0.98x0.95mm_HandSolder, F.Cu at (133.7, 67.7)
- added R6: 100, Resistor_SMD:R_0603_1608Metric_Pad0.98x0.95mm_HandSolder, F.Cu at (133.6, 73.0)
- added R7: 100, Resistor_SMD:R_0603_1608Metric_Pad0.98x0.95mm_HandSolder, F.Cu at (133.6, 78.2)
- added R8: 100, Resistor_SMD:R_0603_1608Metric_Pad0.98x0.95mm_HandSolder, F.Cu at (133.9, 83.3)
- moved D1 74.7 mm to (134.3, 55.6)
- moved D2 74.5 mm to (136.2, 55.6)
- moved D3 74.2 mm to (138.0, 55.6)
- moved D4 74.0 mm to (140.0, 55.6)
- moved R1 66.9 mm to (134.4, 59.5)
- moved R2 66.7 mm to (136.2, 59.5)
- moved R3 66.4 mm to (138.0, 59.5)
- moved R4 66.2 mm to (139.9, 59.4)
Connections:
- J4 pad 22: Net-(J4-Pin_22) -> /LED0
- J6 pad 22: Net-(J4-Pin_22) -> /LED0
- R1 pad 1: /LED2 -> Net-(Q1-C)
- R2 pad 1: /LED3 -> Net-(Q2-C)
- R3 pad 1: /LED1 -> Net-(Q3-C)
- R4 pad 1: Net-(J4-Pin_22) -> Net-(Q4-C)
Routing:
- net /LED1: track 5.10 -> 61.7 mm, vias 0 -> 1
- net /LED0: track 0.00 -> 51.1 mm, vias 0 -> 1
- net /LED2: track 5.08 -> 37.8 mm, vias 0 -> 1
- net Net-(Q4-C): track 0.00 -> 26.1 mm
- net Net-(Q3-C): track 0.00 -> 21.1 mm
- net Net-(Q2-C): track 0.00 -> 15.9 mm
- net +5V: track 5.29 -> 18.8 mm
- net Net-(Q1-C): track 0.00 -> 10.0 mm
- net GND: track 25.4 -> 32.8 mm, vias 0 -> 4
- net /LED3: track 5.08 -> 12.4 mm
- net Net-(J4-Pin_22): track 5.08 -> 0.00 mm
- net Net-(D2-K): track 0.00 -> 2.12 mm
- net Net-(D3-K): track 0.00 -> 2.12 mm
- net Net-(D1-K): track 0.00 -> 2.12 mm
- net Net-(D4-K): track 0.00 -> 2.08 mm
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- added copper zone on In2.Cu, net +1.8V_MCU
- added copper zone on In1.Cu, net GND
Other:
- board size 80 x 82.1 mm -> 80 x 70 mm
